File: Platform/EAGLE/DoorchimeCR2.brd (EAGLE design)
At the start: 60 x 53 mm, 42 parts, among them IC1 STM32G4xx, IC2 7805, IC3 MAX98357A, IC5 78L33F

Commit message: Updated the EAGLE files to include the optional volume pot Updated the Gerbers
Parts:
- added R3: 10K, rcl:RTRIM3339P
- !SD_MODE, +5V, GND, I2S_CK, I2S_SD, I2S_WS, NRST, SWCLK, SWDIO, VDD: value PTR1TP10R -> PTR1TP15R; device testpad:TP10R -> testpad:TP15R
- moved !SD_MODE 1.28 mm to (35.9, 29.1)
- moved I2S_CK 0.64 mm to (25.2, 37.1)
- moved SWDIO 0.64 mm to (23.2, 18.8)
- moved SWCLK 0.32 mm to (28.6, 21.6)
- moved I2S_SD 0.32 mm to (33.0, 32.7)
Connections:
- new net VOLUME_REF: IC1.PF0-OSC_IN, R3.2
- net GND: now also R3.1
- net VDD: now also R3.3
Routing:
- net VOLUME_REF: track 0.00 -> 25.3 mm, vias 0 -> 1
- net VDD: track 49.4 -> 51.5 mm
- net VIN+: track 91.7 -> 92.7 mm
- net !SD_MODE: track 19.5 -> 20.2 mm
- net I2S_CK: track 27.3 -> 28.0 mm
- net SWDIO: track 21.0 -> 21.6 mm
Other:
- board text added: "70-0350 Rev D"
- board text added: "VOL"
- board text removed: "70-0350 Rev C"
