File: Platform/EAGLE/DoorchimeCR2.sch (EAGLE design)
At the start: 42 parts, among them IC1 STM32G4xx, IC2 7805, IC3 MAX98357A, IC5 78L33F

Commit message: Updated the EAGLE files to include the optional volume pot Updated the Gerbers
Parts:
- added R3: 10K, rcl:R-TRIMM3339P
- !SD_MODE, +5V, GND, I2S_CK, I2S_SD, I2S_WS, NRST, SWCLK, SWDIO, VDD: value PTR1TP10R -> PTR1TP15R; device testpad:PTR1TP10R -> testpad:PTR1TP15R
Connections:
- new net VOLUME_REF: IC1.PF0-OSC_IN, R3.S
- net GND: now also R3.E
- net VDD: now also R3.A
Other:
- note added: "OPTIONAL VOLUME POT"
- moved on the sheet: R10, TRIG-1, TRIG-2
